File: atxmega32a4u/pcb/xmega32A4U.brd (EAGLE design)
At the start: 51.8 x 18.8 mm, 23 parts

Commit message: V1.4 production scripts set, boards sent to Seeed and Smart Prototyping
Parts:
- C1, C3: device SparkFun-Capacitors:0603-CAP -> JCM-Capacitors:0603-CAP
- C4, C5, C6, C7, C8: device SparkFun-Capacitors:0402-CAP -> JCM-Capacitors:0402-CAP
- JP1: value M20 -> M191X19; device SparkFun-Connectors:1X20 -> SparkFun-Connectors:1X19
- R1, R3: device SparkFun-Passives:0603-RES -> JCM-Resistors:0603-RES
- R2: device SparkFun-Resistors:0402-RES -> JCM-Resistors:0402-RES
- UC: value XMEGA-A4UVQFN -> XMEGA-A4UVQFN-NP; device JCM:QFN44 -> JCM-IC:QFN44-NOPAD
- moved U$6 18.9 mm to (35.2, 9.96)
- moved R2 2.12 mm to (40.8, 9.14), turned to 90 degrees
- moved U$4 1.68 mm to (43.4, 9.96)
- moved C8 1.49 mm to (40.8, 11.7), turned to 270 degrees
- moved C2 0.76 mm to (38.6, 9.91)
- moved U1 0.51 mm to (35.3, 9.91)
- moved C1 0.10 mm to (39.9, 13.7)
Connections:
- net PDI-DATA: no longer JP1.16
- net PE0: now also JP1.19; no longer JP1.20
- net PE1: now also JP1.18; no longer JP1.19
- net PE2: now also JP1.17; no longer JP1.18
- net PE3: now also JP1.16; no longer JP1.17
Routing:
- net PDI-DATA: track 36.2 -> 18.0 mm
- net 5VINT: track 25.1 -> 30.2 mm
- net PE2: track 22.1 -> 19.9 mm
- net PE0: track 31.9 -> 29.7 mm
- net PE1: track 27.9 -> 25.8 mm
- net PE3: track 19.4 -> 17.2 mm
- net SHLD: track 4.45 -> 5.59 mm
- net 3.3V: track 72.0 -> 72.9 mm
- net PD7/D+: track 22.9 -> 23.6 mm
- net PD6/D-: track 23.2 -> 23.8 mm
- net RST: track 37.4 -> 38.0 mm
- net N$3: track 2.15 -> 1.64 mm
- net 5V: track 7.96 -> 8.44 mm, vias 1 -> 0
- net GND: track 14.2 -> 14.1 mm, vias 19 -> 21
Other:
- board size 51.8 x 18.8 mm -> 49.9 x 18.8 mm
- board text added: "E0"
- board text added: "E1"
- board text added: "E2"
- board text added: "E3"
- board text added: "v0.4"
- board text removed: "PDI-D"
- board text removed: "PE0"
- board text removed: "PE1"
- board text removed: "PE2"
- board text removed: "PE3"
- board text removed: "v0.3"

Commit message: CY8C4245LQI breakout added
Parts:
- U$7: device JCM:AVR_50MIL_PROG -> JCM-Connectors:AVR_50MIL_PROG
Routing:
- net GND: track 14.1 -> 13.5 mm
