File: atxmega32a4u/pcb/xmega32A4U.sch (EAGLE design)
At the start: 22 parts

Commit message: V1.4 production scripts set, boards sent to Seeed and Smart Prototyping
Parts:
- C1, C3: device SparkFun-Capacitors:CAP0603-CAP -> JCM-Capacitors:CAP0603-CAP
- C4, C5, C6, C7, C8: device SparkFun-Capacitors:CAP0402-CAP -> JCM-Capacitors:CAP0402-CAP
- JP1: value M20 -> M191X19; device SparkFun-Connectors:M20 -> SparkFun-Connectors:M191X19
- R1, R3: device SparkFun-Passives:RESISTOR0603-RES -> JCM-Resistors:RESISTOR0603-RES
- R2: device SparkFun-Resistors:RESISTOR0402-RES -> JCM-Resistors:RESISTOR0402-RES
- UC: value XMEGA-A4UVQFN -> XMEGA-A4UVQFN-NP; device JCM:XMEGA-A4UVQFN -> JCM-IC:XMEGA-A4UVQFN-NP
Connections:
- net PDI-DATA: no longer JP1.16
- net PE0: now also JP1.19; no longer JP1.20
- net PE1: now also JP1.18; no longer JP1.19
- net PE2: now also JP1.17; no longer JP1.18
- net PE3: now also JP1.16; no longer JP1.17
Other:
- note added: "v0.4"
- note removed: "v0.3"
Changed lines of the file:
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@@
 <part name="GND2" library="SparkFun-Aesthetics" deviceset="GND" device=""/>
 <part name="U$2" library="SparkFun-Aesthetics" deviceset="5V" device=""/>
-<part name="C1" library="SparkFun-Capacitors" deviceset="CAP" device="0603-CAP" value="1uF">
+<part name="C1" library="JCM-Capacitors" deviceset="CAP" device="0603-CAP" value="1uF">
 <attribute name="PARTNO" value="C0603C105K3PACTU"/>
 </part>
@@
 <part name="P+4" library="SparkFun-Aesthetics" deviceset="3.3V" device=""/>
 <part name="U$3" library="SparkFun-Aesthetics" deviceset="5V" device=""/>
-<part name="C4" library="SparkFun-Capacitors" deviceset="CAP" device="0402-CAP" value="0.1uF">
+<part name="C4" library="JCM-Capacitors" deviceset="CAP" device="0402-CAP" value="0.1uF">
 <attribute name="PARTNO" value="GMK105BJ104KV-F"/>
 </part>
@@
 <attribute name="PARTNO" value="MIC5219-3.3YM5 TR"/>
 </part>
-<part name="R1" library="SparkFun-Passives" deviceset="RESISTOR" device="0603-RES" value="1k">
+<part name="R1" library="JCM-Resistors" deviceset="RESISTOR" device="0603-RES" value="1k">
 <attribute name="PARTNO" value="RC0603FR-071KL"/>
 </part>
@@
 <attribute name="PARTNO" value="68000-418HLF"/>
 </part>
-<part name="C3" library="SparkFun-Capacitors" deviceset="CAP" device="0603-CAP" value="470pF">
+<part name="C3" library="JCM-Capacitors" deviceset="CAP" device="0603-CAP" value="470pF">
 <attribute name="PARTNO" value="C0603C471K5RACTU"/>
 </part>
@@
 <attribute name="PARTNO" value="LTST-C191TBKT"/>
 </part>
-<part name="UC" library="JCM" deviceset="XMEGA-A4U" device="VQFN">
+<part name="UC" library="JCM-IC" deviceset="XMEGA-A4U" device="VQFN-NP" value="XMEGA-A4UVQFN-NP">
 <attribute name="PARTNO" value="ATXMEGA32A4U-MH"/>
 </part>
-<part name="JP1" library="SparkFun-Connectors" deviceset="M20" device="" value="M20">
+<part name="JP1" library="SparkFun-Connectors" deviceset="M19" device="1X19" value="M191X19">
 <attribute name="PARTNO" value="M20-9732046"/>
 </part>
-<part name="C5" library="SparkFun-Capacitors" deviceset="CAP" device="0402-CAP" value="0.1uF">
+<part name="C5" library="JCM-Capacitors" deviceset="CAP" device="0402-CAP" value="0.1uF">
 <attribute name="PARTNO" value="GMK105BJ104KV-F"/>
 </part>
-<part name="C6" library="SparkFun-Capacitors" deviceset="CAP" device="0402-CAP" value="0.1uF">
+<part name="C6" library="JCM-Capacitors" deviceset="CAP" device="0402-CAP" value="0.1uF">
 <attribute name="PARTNO" value="GMK105BJ104KV-F"/>
 </part>
@@
 <attribute name="PARTNO" value="UX60-MB-5S8"/>
 </part>
-<part name="C8" library="SparkFun-Capacitors" deviceset="CAP" device="0402-CAP" value="4.7nF">
+<part name="C8" library="JCM-Capacitors" deviceset="CAP" device="0402-CAP" value="4.7nF">
 <attribute name="PARTNO" value="C0402C472K3RACTU"/>
 </part>
-<part name="R2" library="SparkFun-Resistors" deviceset="RESISTOR" device="0402-RES" value="1M">
+<part name="R2" library="JCM-Resistors" deviceset="RESISTOR" device="0402-RES" value="1M">
 <attribute name="PARTNO" value="CRCW04021M00JNED"/>
 </part>
 <part name="SHLD" library="Power or GND " deviceset="GND_EARTH" device=""/>
-<part name="C7" library="SparkFun-Capacitors" deviceset="CAP" device="0402-CAP" value="0.1uF">
+<part name="C7" library="JCM-Capacitors" deviceset="CAP" device="0402-CAP" value="0.1uF">
 <attribute name="PARTNO" value="GMK105BJ104KV-F"/>
 </part>
@@
 <attribute name="PARTNO" value="CG0603MLC-05E"/>
 </part>
-<part name="R3" library="SparkFun-Passives" deviceset="RESISTOR" device="0603-RES" value="1k">
+<part name="R3" library="JCM-Resistors" deviceset="RESISTOR" device="0603-RES" value="1k">
 <attribute name="PARTNO" value="RC0603FR-071KL"/>
 </part>
@@
 <text x="162.56" y="-35.56" size="1.778" layer="94">USB Connector</text>
 <text x="182.88" y="-66.04" size="2.54" layer="97">Joseph Moreland</text>
-<text x="248.92" y="-66.04" size="2.54" layer="97">v0.3</text>
+<text x="248.92" y="-66.04" size="2.54" layer="97">v0.4</text>
 <wire x1="86.36" y1="-73.66" x2="86.36" y2="-2.54" width="0.3048" layer="94"/>
 <wire x1="160.02" y1="40.64" x2="160.02" y2="111.76" width="0.3048" layer="94"/>
@@
 <attribute name="PARTNO" x="73.66" y="66.04" size="1.778" layer="96" display="off"/>
 </instance>
-<instance part="JP1" gate="G$1" x="40.64" y="-7.62" rot="R180">
-<attribute name="PARTNO" x="40.64" y="-7.62" size="1.778" layer="96" display="off"/>
+<instance part="JP1" gate="G$1" x="40.64" y="-35.56" rot="R180">
+<attribute name="PARTNO" x="40.64" y="-35.56" size="1.778" layer="96" display="off"/>
 </instance>
 <instance part="C5" gate="G$1" x="200.66" y="99.06">
@@
 </segment>
 <segment>
+<wire x1="30.48" y1="-50.8" x2="20.32" y2="-50.8" width="0.1524" layer="91"/>
+<label x="20.32" y="-50.8" size="1.778" layer="95"/>
+<pinref part="JP1" gate="G$1" pin="16"/>
+</segment>
+</net>
+<net name="PE2" class="0">
+<segment>
+<wire x1="114.3" y1="71.12" x2="127" y2="71.12" width="0.1524" layer="91"/>
+<label x="121.92" y="71.12" size="1.778" layer="95"/>
+<pinref part="UC" gate="G$1" pin="PE2(OC0C/RXD0)"/>
+</segment>
+<segment>
 <wire x1="30.48" y1="-53.34" x2="20.32" y2="-53.34" width="0.1524" layer="91"/>
 <label x="20.32" y="-53.34" size="1.778" layer="95"/>
@@
 </segment>
 </net>
-<net name="PE2" class="0">
-<segment>
-<wire x1="114.3" y1="71.12" x2="127" y2="71.12" width="0.1524" layer="91"/>
-<label x="121.92" y="71.12" size="1.778" layer="95"/>
-<pinref part="UC" gate="G$1" pin="PE2(OC0C/RXD0)"/>
+<net name="PE1" class="0">
+<segment>
+<wire x1="114.3" y1="73.66" x2="127" y2="73.66" width="0.1524" layer="91"/>
+<label x="121.92" y="73.66" size="1.778" layer="95"/>
+<pinref part="UC" gate="G$1" pin="PE1(OC0B/XCK0/SCL)"/>
 </segment>
 <segment>
@@
 </segment>
 </net>
-<net name="PE1" class="0">
-<segment>
-<wire x1="114.3" y1="73.66" x2="127" y2="73.66" width="0.1524" layer="91"/>
-<label x="121.92" y="73.66" size="1.778" layer="95"/>
-<pinref part="UC" gate="G$1" pin="PE1(OC0B/XCK0/SCL)"/>
+<net name="PE0" class="0">
+<segment>
+<wire x1="114.3" y1="76.2" x2="127" y2="76.2" width="0.1524" layer="91"/>
+<label x="121.92" y="76.2" size="1.778" layer="95"/>
+<pinref part="UC" gate="G$1" pin="PE0(OC0A/SDA)"/>
 </segment>
 <segment>
@@
 <label x="20.32" y="-58.42" size="1.778" layer="95"/>
 <pinref part="JP1" gate="G$1" pin="19"/>
-</segment>
-</net>
-<net name="PE0" class="0">
-<segment>
-<wire x1="114.3" y1="76.2" x2="127" y2="76.2" width="0.1524" layer="91"/>
-<label x="121.92" y="76.2" size="1.778" layer="95"/>
-<pinref part="UC" gate="G$1" pin="PE0(OC0A/SDA)"/>
-</segment>
-<segment>
-<wire x1="30.48" y1="-60.96" x2="20.32" y2="-60.96" width="0.1524" layer="91"/>
-<label x="20.32" y="-60.96" size="1.778" layer="95"/>
-<pinref part="JP1" gate="G$1" pin="20"/>
 </segment>
 </net>
@@
 </segment>
 <segment>
-<wire x1="30.48" y1="-50.8" x2="20.32" y2="-50.8" width="0.1524" layer="91"/>
-<label x="20.32" y="-50.8" size="1.778" layer="95"/>
-<pinref part="JP1" gate="G$1" pin="16"/>
-</segment>
-<segment>

Commit message: CY8C4245LQI breakout added
Parts:
- U$7: device JCM:AVR_PDI_PROG -> JCM-Connectors:AVR_PDI_PROG
Changed lines of the file:
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@@
 <?xml version="1.0" encoding="utf-8"?>
 <!DOCTYPE eagle SYSTEM "eagle.dtd">
-<eagle version="6.4">
+<eagle version="6.5.0">
 <drawing>
 <settings>
@@
 <layers>
 <layer number="1" name="Top" color="4" fill="1" visible="no" active="no"/>
+<layer number="2" name="Route2" color="1" fill="3" visible="no" active="no"/>
+<layer number="3" name="Route3" color="4" fill="3" visible="no" active="no"/>
+<layer number="4" name="Route4" color="1" fill="4" visible="no" active="no"/>
+<layer number="5" name="Route5" color="4" fill="4" visible="no" active="no"/>
+<layer number="6" name="Route6" color="1" fill="8" visible="no" active="no"/>
+<layer number="7" name="Route7" color="4" fill="8" visible="no" active="no"/>
+<layer number="8" name="Route8" color="1" fill="2" visible="no" active="no"/>
+<layer number="9" name="Route9" color="4" fill="2" visible="no" active="no"/>
+<layer number="10" name="Route10" color="1" fill="7" visible="no" active="no"/>
+<layer number="11" name="Route11" color="4" fill="7" visible="no" active="no"/>
+<layer number="12" name="Route12" color="1" fill="5" visible="no" active="no"/>
+<layer number="13" name="Route13" color="4" fill="5" visible="no" active="no"/>
+<layer number="14" name="Route14" color="1" fill="6" visible="no" active="no"/>
+<layer number="15" name="Route15" color="4" fill="6" visible="no" active="no"/>
 <layer number="16" name="Bottom" color="1" fill="1" visible="no" active="no"/>
 <layer number="17" name="Pads" color="2" fill="1" visible="no" active="no"/>
@@
 <attribute name="PARTNO" value="LTST-C190KGKT"/>
 </part>
-<part name="U$7" library="JCM" deviceset="AVR_PDI_PROG" device="">
+<part name="U$7" library="JCM-Connectors" deviceset="AVR_PDI_PROG" device="">
 <attribute name="PARTNO" value="LPPB032NFSP-RC"/>
 </part>
